Commit message: Fix base link to world link in arch_loboot_urdf; debug detectFun() in process_sherds.py

File: for_pyrobot/locobot_description/arch_locobot_description.urdf (robot description, URDF)
Before this commit: robot locobot, 26 links, 25 joints
Links:
- link cam_mount: mass 2.091937 -> 0.001; geometry collision mesh filename=package://locobot_description/meshes/interbotix_cam_mount.S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 scale=0.001 0.001 0.001; visual cylinder length=0.001 radius=.0001
- link head_pan_link: mass 0.0182769203076134 -> 0.001; geometry collision mesh filename=package://locobot_description/meshes/tilt_link.STL; visual cylinder length=0.001 radius=.0001
- link head_tilt_link: mass 0.0547677687275323 -> 0.001; geometry collision mesh filename=package://locobot_description/meshes/roll_link.STL; visual cylinder length=0.001 radius=.0001

Commit message: reduced camera_link mass and moments; add friction to gripper finger link; static transform between world and base_footprint. stop work for 5/29

File: for_pyrobot/locobot_description/arch_locobot_description.urdf (robot description, URDF)
Before this commit: robot locobot, 26 links, 25 joints
Links:
- added link world
- link camera_link: mass 0.0381925651163644 -> 0.000381925651163644
Joints:
- added joint fixed: type fixed, parent world, child base_footprint, origin xyz=0 0 0 rpy=0 0 0

Commit message: mu and mu2 friction = 1.0 on gripper fingers

File: for_pyrobot/locobot_description/arch_locobot_description.urdf (robot description, URDF)
Before this commit: robot locobot, 27 links, 26 joints
Joints:
- joint camera_joint: origin xyz=0.04 0 0.055 rpy=0 0 0 -> xyz=0.04 0.0 0.055 rpy=0 0 0
