Commit message: Update simulation   -Modify some launch files to use our updated urdf   -Remove pan and tilt joint entirely from the simulation   -Add local copies of all relevant pyrobot launch files that needed updating (in future, perhaps we should fork pyrobot)   -Add gazebo_locobot_control executable to remove pan and tilt joints   -Update our launch files to include correct location of launch files   -Include perception inside of archaeology.launch

File: urdf/arch_locobot_description.urdf (robot description, URDF)
Before this commit: robot locobot, 27 links, 26 joints
Links:
- removed link cam_mount
- removed link head_pan_link
- removed link head_tilt_link
Joints:
- removed joint cam_mount_joint
- removed joint head_pan_joint
- removed joint head_tilt_joint

Commit message: comment out ar_tag link and joint

File: urdf/arch_locobot_description.urdf (robot description, URDF)
Before this commit: robot locobot, 24 links, 23 joints
Links:
- removed link ar_tag
Joints:
- removed joint ar_tag_joint

Commit message: fix base_footprint to mat_link instead of world

File: urdf/arch_locobot_description.urdf (robot description, URDF)
Before this commit: robot locobot, 23 links, 22 joints
Links:
- removed link world
- added link mat_link
Joints:
- joint fixed: origin xyz=0 0 0 rpy=0 0 0 -> xyz=0 0 0.0025 rpy=0 0 0; parent world -> mat_link

Commit message: comment out fixed joint between base_footprint and mat_link - locobot no longer jittering, it seems

File: urdf/arch_locobot_description.urdf (robot description, URDF)
Before this commit: robot locobot, 23 links, 22 joints
Links:
- removed link mat_link
Joints:
- removed joint fixed

Commit message: turn fixed joint for locobot back on

File: urdf/arch_locobot_description.urdf (robot description, URDF)
Before this commit: robot locobot, 22 links, 21 joints
Links:
- added link mat_link
Joints:
- added joint fixed: type fixed, parent mat_link, child base_footprint, origin xyz=0 0 0.0025 rpy=0 0 0

Commit message: fix base_footprint to world_link

File: urdf/arch_locobot_description.urdf (robot description, URDF)
Before this commit: robot locobot, 23 links, 22 joints
Links:
- removed link mat_link
- added link world_link
Joints:
- joint fixed: parent mat_link -> world_link

Commit message: fix typo in fixed joint between world and base_footprint

File: urdf/arch_locobot_description.urdf (robot description, URDF)
Before this commit: robot locobot, 23 links, 22 joints
Links:
- removed link world_link
- added link world
Joints:
- joint fixed: parent world_link -> world

Commit message: Update setup to be more like final use case   -Make sherd mat same size as standard folding table   -Allow base joint to rotateall the way around   -Update mat layout and world file     --Pickup area to left of arm     --Scale directly in front     --Camera front and right     --Discard area to right   -Shrink horizontal arm for camera mount   -Increase camera resolution to 4K   -Update gazebo grip parameters to make grasping more reliable   -Fix typo in sherd_states

File: urdf/arch_locobot_description.urdf (robot description, URDF)
Before this commit: robot locobot, 23 links, 22 joints
Joints:
- joint joint_1: limit lower=-1.57 upper=1.57 effort=10 velocity=1 -> lower=-3.14 upper=3.14 effort=10 velocity=1
